File: circuit/gen2/7seg_led.kicad_sch (KiCad schematic)
At the start: 26 parts, among them Q1 2SC1815, Q2 2SC1815, Q3 2SC1815, Q4 2SC1815, Q5 2SC1815, U2 4digit_7seg_led

Commit message: [update] gen2 is production ready
Parts:
- removed 10k2, 10k3, 10k4, 270Ω2, 270Ω3, 270Ω4, 270Ω5, 270Ω6: R_US, Resistor_THT:R_Axial_DIN0207_L6.3mm_D2.5mm_P10.16mm_Horizontal, symbol Device:R_US
- added R_US10, R_US11, R_US9: 10k, Resistor_SMD:R_0805_2012Metric, symbol Device:R_US
- added R_US2, R_US3, R_US4, R_US5, R_US6: 270, Resistor_SMD:R_0805_2012Metric, symbol Device:R_US
- LED1: renamed from GREEN1; value LED -> GREEN; footprint LED_THT:LED_D1.8mm_W1.8mm_H2.4mm_Horizontal_O1.27mm_Z1.6mm -> LED_THT:LED_D5.0mm
- LED2: renamed from YELLOW1; value LED -> YELLOW; footprint LED_THT:LED_D1.8mm_W1.8mm_H2.4mm_Horizontal_O1.27mm_Z1.6mm -> LED_THT:LED_D5.0mm
- LED3: renamed from RED1; value LED -> RED; footprint LED_THT:LED_D1.8mm_W1.8mm_H2.4mm_Horizontal_O1.27mm_Z1.6mm -> LED_THT:LED_D5.0mm
- Q1, Q2, Q3, Q4, Q5: footprint Package_TO_SOT_THT:TO-92_Inline_Wide -> Package_TO_SOT_SMD:SOT-23
- R_US1: renamed from 270Ω1; value R_US -> 270; footprint Resistor_THT:R_Axial_DIN0207_L6.3mm_D2.5mm_P10.16mm_Horizontal -> Resistor_SMD:R_0805_2012Metric
- R_US12: renamed from 10k5; value R_US -> 10k; footprint Resistor_THT:R_Axial_DIN0207_L6.3mm_D2.5mm_P10.16mm_Horizontal -> Resistor_SMD:R_0805_2012Metric
- R_US13: renamed from 270Ω8; value R_US -> 270; footprint Resistor_THT:R_Axial_DIN0207_L6.3mm_D2.5mm_P10.16mm_Horizontal -> Resistor_SMD:R_0805_2012Metric
- R_US14: renamed from 270Ω9; value R_US -> 270; footprint Resistor_THT:R_Axial_DIN0207_L6.3mm_D2.5mm_P10.16mm_Horizontal -> Resistor_SMD:R_0805_2012Metric
- R_US15: renamed from 270Ω10; value R_US -> 270; footprint Resistor_THT:R_Axial_DIN0207_L6.3mm_D2.5mm_P10.16mm_Horizontal -> Resistor_SMD:R_0805_2012Metric
- R_US7: renamed from 270Ω7; value R_US -> 270; footprint Resistor_THT:R_Axial_DIN0207_L6.3mm_D2.5mm_P10.16mm_Horizontal -> Resistor_SMD:R_0805_2012Metric
- R_US8: renamed from 10k1; value R_US -> 10k; footprint Resistor_THT:R_Axial_DIN0207_L6.3mm_D2.5mm_P10.16mm_Horizontal -> Resistor_SMD:R_0805_2012Metric
- U2: value 4digit_7seg_led -> OSL_40391_LRA
- primary1, secondary1: footprint Package_DIP:DIP-16_W7.62mm_Socket -> Package_SO:SOIC-16_3.9x9.9mm_P1.27mm
Connections:
- net GNDPWR: now also Q1.2 (E), Q2.2 (E), Q3.2 (E), Q4.2 (E), Q5.2 (E); no longer Q1.1 (E), Q2.1 (E), Q3.1 (E), Q4.1 (E), Q5.1 (E)
- net at Q5.3 (C): now also U2.1 (CC1)
- net at primary1.1 (QB): now also R_US9.2
- net at U2.8 (CC4): now also Q2.3 (C); no longer Q2.2 (C)
- net at R_US12.1: now also Q2.1 (B); no longer Q2.3 (B)
- net at primary1.2 (QC): now also R_US10.2
- net at primary1.3 (QD): now also R_US11.2
- net at Q4.3 (C): now also U2.2 (CC2)
- net at Q3.3 (C): now also U2.6 (CC3)
- net at secondary1.2 (QC): now also R_US2.2
- net at secondary1.3 (QD): now also R_US3.2
- net at secondary1.4 (QE): now also R_US4.2
- net at secondary1.5 (QF): now also R_US5.2
- net at secondary1.6 (QG): now also R_US6.2
- net at U2.5 (e): now also R_US3.1
- net at R_US8.1: now also Q1.1 (B); no longer Q1.3 (B)
- net at U2.13 (c/D3): now also R_US5.1
- net at U2.16 (b/D2): now also R_US6.1
- net at U2.11 (f): now also R_US2.1
- net at U2.3 (d): now also R_US4.1
- net at U2.4 (CC5): now also Q1.3 (C); no longer Q1.2 (C)
- new net: Q4.1 (B), R_US10.1
- new net: Q3.1 (B), R_US11.1
- new net: Q5.1 (B), R_US9.1
