File: circuit/gen2/gen2.kicad_sch (KiCad schematic)
At the start: 5 parts, among them J1 Conn_01x02_Socket, J2 Conn_02x20_Row_Letter_Last, J3 Conn_01x02_Socket, J4 Conn_02x20_Row_Letter_Last, U1 ESP32-DevKitC

Commit message: [update] gen2 is production ready
Parts:
- J1, J3: footprint Connector_PinHeader_2.54mm:PinHeader_1x02_P2.54mm_Vertical -> Connector_JST:JST_XH_S2B-XH-A_1x02_P2.50mm_Horizontal
Connections:
- net +5V: now also J3.2 (Pin_2); no longer J3.1 (Pin_1)
- net GNDPWR: now also J3.1 (Pin_1); no longer J3.2 (Pin_2)
- new net: J2.none_a (Pin_none_a), J2.none_b (Pin_none_b)
Other:
- sheet pin_button ports: added select_button, start_button; removed button
Changed lines of the file:
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@@
 				)
 			)
-			(property "Footprint" ""
+			(property "Footprint" "MyPartsLibrary:PinSocket_2x20_P2.54mm_1a-19a"
 				(at 0 0 0)
 				(effects
@@
 				)
 			)
-			(property "Description" "Generic connector, double row, 02x20, row letter last pin numbering scheme (pin number consists of a letter for the row and a number for the pin index in this row. 1a, ..., Na; 1b, ..., Nb)), script generated (kicad-library-utils/schlib/autogen/connector/)"
+			(property "Description" ""
 				(at 0 0 0)
 				(effects
@@
 				)
 				(pin passive line
-					(at -5.08 -25.4 0)
-					(length 3.81)
-					(name ""
-						(effects
-							(font
-								(size 1.27 1.27)
-							)
-						)
-					)
-					(number ""
-						(effects
-							(font
-								(size 1.27 1.27)
-							)
-						)
-					)
-				)
-				(pin passive line
-					(at 7.62 -25.4 180)
-					(length 3.81)
-					(name ""
-						(effects
-							(font
-								(size 1.27 1.27)
-							)
-						)
-					)
-					(number ""
-						(effects
-							(font
-								(size 1.27 1.27)
-							)
-						)
-					)
-				)
-				(pin passive line
 					(at -5.08 0 0)
 					(length 3.81)
@@
 					)
 				)
+				(pin passive line
+					(at -5.08 -25.4 0)
+					(length 3.81)
+					(name "Pin_none_a"
+						(effects
+							(font
+								(size 1.27 1.27)
+							)
+						)
+					)
+					(number "none_a"
+						(effects
+							(font
+								(size 1.27 1.27)
+							)
+						)
+					)
+				)
+				(pin passive line
+					(at 7.62 -25.4 180)
+					(length 3.81)
+					(name "Pin_none_b"
+						(effects
+							(font
+								(size 1.27 1.27)
+							)
+						)
+					)
+					(number "none_b"
+						(effects
+							(font
+								(size 1.27 1.27)
+							)
+						)
+					)
+				)
 			)
 		)
@@
 	)
 	(junction
+		(at 172.72 118.11)
+		(diameter 0)
+		(color 0 0 0 0)
+	)
+	(junction
 		(at 172.72 140.97)
 		(diameter 0)
@@
 	)
 	(junction
-		(at 172.72 115.57)
+		(at 172.72 135.89)
 		(diameter 0)
 		(color 0 0 0 0)
 	)
 	(junction
-		(at 172.72 135.89)
+		(at 238.76 99.06)
 		(diameter 0)
 		(color 0 0 0 0)
 	)
 	(junction
-		(at 238.76 99.06)
+		(at 172.72 120.65)
 		(diameter 0)
 		(color 0 0 0 0)
@@
 	(wire
 		(pts
-			(xy 138.43 110.49) (xy 154.94 110.49)
+			(xy 138.43 115.57) (xy 154.94 115.57)
 		)
 		(stroke
@@
 	(wire
 		(pts
-			(xy 138.43 115.57) (xy 172.72 115.57)
+			(xy 138.43 118.11) (xy 172.72 118.11)
 		)
 		(stroke
@@
 	(wire
 		(pts
+			(xy 138.43 120.65) (xy 172.72 120.65)
+		)
+		(stroke
+			(width 0)
+			(type default)
+		)
+	)
+	(wire
+		(pts
 			(xy 298.45 152.4) (xy 311.15 152.4)
 		)
@@
 	(wire
 		(pts
-			(xy 154.94 110.49) (xy 154.94 140.97)
+			(xy 154.94 115.57) (xy 154.94 140.97)
 		)
 		(stroke
@@
 	)
 	(symbol
+		(lib_name "Conn_01x02_Socket_1")
 		(lib_id "Connector:Conn_01x02_Socket")
 		(at 214.63 87.63 270)
@@
 			)
 		)
-		(property "Footprint" "Connector_PinHeader_2.54mm:PinHeader_1x02_P2.54mm_Vertical"
+		(property "Footprint" "Connector_JST:JST_XH_S2B-XH-A_1x02_P2.50mm_Horizontal"
 			(at 214.63 87.63 0)
 			(effects
@@
 		(pin "11b"
 		)
-		(pin ""
+		(pin "none_b"
 		)
 		(pin "1b"
@@
 		(pin "9a"
 		)
-		(pin ""
+		(pin "none_a"
 		)
 		(pin "10b"
@@
 			)
 		)
-		(property "Footprint" "Connector_PinHeader_2.54mm:PinHeader_1x02_P2.54mm_Vertical"
+		(property "Footprint" "Connector_JST:JST_XH_S2B-XH-A_1x02_P2.50mm_Horizontal"
 			(at 168.91 193.04 0)
 			(effects
@@
 	)
 	(sheet
-		(at 116.84 106.68)
-		(size 21.59 12.7)
+		(at 116.84 113.03)
+		(size 21.59 10.16)
 		(fields_autoplaced yes)
 		(stroke
@@
 		)
 		(property "Sheetname" "pin_button"
-			(at 116.84 105.9684 0)
+			(at 116.84 112.3184 0)
 			(effects
 				(font
@@
 		)
 		(property "Sheetfile" "pin_button.kicad_sch"
-			(at 116.84 119.9646 0)
+			(at 116.84 123.7746 0)
 			(effects
 				(font
@@
 			)
 		)
-		(pin "button" input
-			(at 138.43 115.57 0)
+		(pin "start_button" input
+			(at 138.43 118.11 0)
 			(effects
 				(font
@@
 		)
 		(pin "buzzer" input
-			(at 138.43 110.49 0)
+			(at 138.43 115.57 0)
+			(effects
+				(font
+					(size 1.27 1.27)
+				)
+				(justify right)
+			)
+		)
+		(pin "select_button" input
+			(at 138.43 120.65 0)
 			(effects
 				(font
@@
 	)
 	(sheet
-		(at 116.84 125.73)
-		(size 21.59 13.97)
+		(at 116.84 128.27)
+		(size 21.59 10.16)
 		(fields_autoplaced yes)
 		(stroke
@@
 		)
 		(property "Sheetname" "7seg_led"
-			(at 116.84 125.0184 0)
+			(at 116.84 127.5584 0)
 			(effects
 				(font
@@
 		)
 		(property "Sheetfile" "7seg_led.kicad_sch"
-			(at 116.84 140.2846 0)
+			(at 116.84 139.0146 0)
 			(effects
 				(font
