File: circuit/gen2/pin_button.kicad_sch (KiCad schematic)
At the start: 3 parts, among them SW1 SW_Push

Commit message: [update] gen2 is production ready
Parts:
- added R_US16: 10k, Resistor_SMD:R_0805_2012Metric, symbol Device:R_US
- added SW1: select, Button_Switch_SMD:SW_SPST_PTS645, symbol Switch:SW_Push
- BZ1: value Buzzer -> HDB06LFPN
- R_US17: renamed from 10k6; value R_US -> 10k; footprint Resistor_THT:R_Axial_DIN0207_L6.3mm_D2.5mm_P10.16mm_Horizontal -> Resistor_SMD:R_0805_2012Metric
- SW2: renamed from SW1; value SW_Push -> start
Connections:
- net button is gone; now on net buzzer: BZ1.1 (-)
- net +3V3: now also R_US16.2
- net GNDPWR: now also SW2.2, SW1.1; no longer SW2.1
- net buzzer: no longer R_US17.1, SW2.2
- new net select_button: R_US16.1, SW1.2
- new net start_button: R_US17.1, SW2.1
Other:
- moved on the sheet: BZ1, R_US17
