File: circuit/gen3.kicad_pcb (KiCad board)
At the start: 2 copper layers, 100 x 100 mm, 45 parts, among them J1 Jack-DC, J2 Conn_02x20_Row_Letter_Last, J3 Conn_02x20_Row_Letter_Last, J4 Conn_01x02_Socket, J5 Conn_01x02_Socket, Q1 2SC1815, Q2 2SC1815, Q3 2SC1815, Q4 2SC1815, Q5 2SC1815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

Commit message: [update] increase GND track width
Parts:
- J1: footprint Connector_BarrelJack:BarrelJack_CUI_PJ-102AH_Horizontal -> Connector_BarrelJack:BarrelJack_Horizontal
- SW1: footprint MyParts:SW-TH_SS-12F44-G5 -> Button_Switch_THT:SW_Slide_SPDT_Straight_CK_OS102011MS2Q
- turned J1 to 0 degrees
Connections:
- BZ1 pad 1: +3.3V -> +3V3
- D1 pad 1: +3.3V -> +3V3
- J3 pad 36a: /Pin36 -> +3V3
- J3 pad 36b: /Pin36 -> +3V3
- J4 pad 2: /Pin36 -> +3V3
Routing:
- net GNDPWR: track 189.1 -> 22.8 mm, vias 21 -> 23
- net +3V3: track 111.1 -> 250.9 mm, vias 2 -> 4
- net /Pin36: track 44.2 -> 0.00 mm
- net +3.3V: track 21.1 -> 0.00 mm
- net /Pin25: track 66.8 -> 76.0 mm
- net /Pin22: track 90.9 -> 81.8 mm
- net Net-(SW1-B): track 13.8 -> 12.6 mm, vias 1 -> 0
- net /Pin29: track 78.5 -> 79.4 mm
