File: circuit/gen3.kicad_pcb (KiCad board)
At the start: 2 copper layers, 100 x 100 mm, 45 parts, among them J1 Jack-DC, J2 Conn_02x20_Row_Letter_Last, J3 Conn_02x20_Row_Letter_Last, J4 Conn_01x02_Socket, J5 Conn_01x02_Socket, Q1 2SC1815, Q2 2SC1815, Q3 2SC1815, Q4 2SC1815, Q5 2SC1815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

Commit message: [add] generated produciton files
Parts:
- turned R_US1 to 90 degrees
Routing:
- net Net-(LED3-A): track 14.0 -> 9.02 mm, vias 1 -> 0
- net /Pin25: track 76.0 -> 71.1 mm
- net Net-(LED4-A): track 12.8 -> 8.57 mm, vias 1 -> 0
- net Net-(LED2-A): track 12.7 -> 8.53 mm, vias 1 -> 0
- net +3V3: track 250.9 -> 254.8 mm, vias 4 -> 3
- net /7seg_led/DP: track 79.0 -> 75.5 mm
- net Net-(U1-QG): track 114.4 -> 111.2 mm
- net Net-(U2-QD): track 13.7 -> 10.7 mm
- net Net-(U1-QH): track 94.6 -> 93.5 mm
- net Net-(U2-QA): track 13.6 -> 13.0 mm
- net GNDPWR: vias 23 -> 28
